Commit message: vehicle working

File: turtlebot3_ignition/urdf/vehicle.urdf (robot description, URDF)
Before this commit: robot vehicle, 15 links, 14 joints
Links:
- removed link left_wheel
- removed link right_wheel
- removed link sensor/air_pressure
- removed link sensor/altimeter
- removed link sensor/camera
- removed link sensor/depth_camera
- removed link sensor/force_torque
- removed link sensor/magnetometer
- removed link sensor/rgbd_camera
- removed link sensor/thermal_camera
Joints:
- removed joint air_pressure_joint
- removed joint altimeter_joint
- removed joint camera_joint
- removed joint depth_camera_joint
- removed joint force_torque_joint
- removed joint left_wheel_joint
- removed joint magnetometer_joint
- removed joint rgbd_camera_joint
- removed joint right_wheel_joint
- removed joint thermal_camera_joint
